File: KiCAD/aviationAirportLEDMap/aviationAirportLEDMap.kicad_sch (KiCad schematic)
At the start: 0 parts

Commit message: first attempt at schematic, added a few symbols for pi zero w, pwr connections and the LED's.
added *.bak to the .gitignore as they aren't needed  for tracking.
Parts:
- added C1: 500-1000 uF, symbol Device:C_Small_US
- added D2: 1N5822, Diode_THT:D_DO-201AD_P15.24mm_Horizontal, symbol Diode:1N5822
- added F1: FAST BLOW 2.5A-250V FUSE, symbol Device:Fuse
- added LED1: KSPK, symbol adafruitHardware:NEOPIXEL_MINI_BUTTON_PCB
- added LED2: KPVU, symbol adafruitHardware:NEOPIXEL_MINI_BUTTON_PCB
- added LED3: KSLC, symbol adafruitHardware:NEOPIXEL_MINI_BUTTON_PCB
- added LED4: KTVY, symbol adafruitHardware:NEOPIXEL_MINI_BUTTON_PCB
- added LED5: KENV, symbol adafruitHardware:NEOPIXEL_MINI_BUTTON_PCB
- added LED6: KHIF, symbol adafruitHardware:NEOPIXEL_MINI_BUTTON_PCB
- added LED7: KOGD, symbol adafruitHardware:NEOPIXEL_MINI_BUTTON_PCB
- added LED8: KBMC, symbol adafruitHardware:NEOPIXEL_MINI_BUTTON_PCB
- added LED9: KLGU, symbol adafruitHardware:NEOPIXEL_MINI_BUTTON_PCB
- added PI1: MAIN CONTROLLER, symbol raspberryPI:Raspberry_Pi_Zero_W
- added PWR1: 5VDC - 10A, symbol commonHardware:5VDC_10A_PWR_SUPPLY
- added PWR_ADAPTOR1: (no value), symbol adafruitHardware:2.1mm_BARREL_JACK_PWR_ADAPTOR
- added R1: 300-900Ω, symbol Device:R_US
Connections:
- new net: C1.1, D2.2 (A), PWR_ADAPTOR1. (-PWR)
- new net: C1.2, LED1.3 (+5V)
- new net: LED6.4 (GND), LED7.1 (GND)
- new net: LED6.5 (DO), LED7.2 (DIN)
- new net: LED6.6 (+5V), LED7.3 (+5V)
- new net: LED1.1 (GND), PI1.6 (GND), PWR_ADAPTOR1. (-PWR)
- new net: LED1.2 (DIN), R1.2
- new net: F1.1, PI1.2 (5VDC)
- new net: D2.1 (K), F1.2
- new net: PWR1. (-5VDC), PWR_ADAPTOR1.1 (+PWR_PIN)
- new net: PWR1. (-5VDC), PWR_ADAPTOR1.2 (-PWR_JACKET)
- new net: PI1.18 (GPIO24), R1.1
- new net GRD IN: PWR1.3 (GND)
- new net LINE IN: LED1.4 (GND), LED2.1 (GND), LED2.4 (GND), LED3.1 (GND), LED3.4 (GND), LED4.1 (GND), LED4.4 (GND), LED5.1 (GND), LED5.4 (GND), LED6.1 (GND), LED7.4 (GND), LED8.1 (GND), LED8.4 (GND), LED9.1 (GND), PWR1.1 (LINE)
- new net NEUTRAL IN: LED1.5 (DO), LED2.2 (DIN), LED2.5 (DO), LED3.2 (DIN), LED3.5 (DO), LED4.2 (DIN), LED4.5 (DO), LED5.2 (DIN), LED5.5 (DO), LED6.2 (DIN), LED7.5 (DO), LED8.2 (DIN), LED8.5 (DO), LED9.2 (DIN), PWR1.2 (NEUTRAL)
- new net RED: LED1.6 (+5V), LED2.3 (+5V), LED2.6 (+5V), LED3.3 (+5V), LED3.6 (+5V), LED4.3 (+5V), LED4.6 (+5V), LED5.3 (+5V), LED5.6 (+5V), LED6.3 (+5V), LED7.6 (+5V), LED8.3 (+5V), LED8.6 (+5V), LED9.3 (+5V)
Other:
- note added: "2.1mm BARREL JACK CABLE"
- title: (none) -> SALT LAKE VALLEY LED MAP

Commit message: cleaned up the schematic a bit.
Parts:
- added J1, J2: Screw_Terminal_01x03, symbol Connector:Screw_Terminal_01x03
- added LED10: LGU, symbol adafruitHardware:NEOPIXEL_MINI_BUTTON_PCB
- added LED11: KEVW, symbol adafruitHardware:NEOPIXEL_MINI_BUTTON_PCB
- LED1: value KSPK -> KHCR
- LED3: value KSLC -> KSVR
- LED4: value KTVY -> KSLC
- LED5: value KENV -> KTVY
- LED6: value KHIF -> KENV
- LED7: value KOGD -> KHIF
- LED8: value KBMC -> KOGD
- LED9: value KLGU -> KBMC
- PI1: value MAIN CONTROLLER -> RASPBERRY PI ZERO W
- PWR_ADAPTOR1: value (none) -> 2.1mm BARREL JACK PORT - SOLDERED TO THROUGH BOARD
Connections:
- net LINE IN: now also LED6.4 (GND), LED7.1 (GND), LED9.4 (GND), LED10.1 (GND); no longer LED5.4 (GND), LED6.1 (GND)
- net NEUTRAL IN: now also LED6.5 (DO), LED7.2 (DIN), LED9.5 (DO), LED10.2 (DIN); no longer LED5.5 (DO), LED6.2 (DIN)
- net RED: now also LED6.6 (+5V), LED7.3 (+5V), LED9.6 (+5V), LED10.3 (+5V); no longer LED5.6 (+5V), LED6.3 (+5V)
- net at D2.2 (A), PWR_ADAPTOR1. (-PWR): now also C1.2; no longer C1.1
- net at LED1.3 (+5V): now also J1.6 (Pin_1); no longer C1.2
- net at R1.2: now also J1.2 (Pin_2); no longer LED1.2 (DIN)
- net at PI1.2 (5VDC): now also J2.3 (Pin_3); no longer F1.1
- net at F1.2: now also J2.6 (Pin_1); no longer D2.1 (K)
- net at R1.1: now also J2.5 (Pin_1); no longer PI1.18 (GPIO24)
- net at PI1.12 (GPIO18): now also J2.2 (Pin_2)
- new net: J1.1 (Pin_1), J2.4 (Pin_1), PWR_ADAPTOR1. (-PWR)
- new net: C1.1, J1.3 (Pin_3)
- new net: J1.4 (Pin_1), LED1.1 (GND)
- new net: J1.5 (Pin_1), LED1.2 (DIN)
- new net: J2.1 (Pin_1), PI1.6 (GND)
- new net: LED10.4 (GND), LED11.1 (GND)
- new net: LED10.5 (DO), LED11.2 (DIN)
- new net: LED10.6 (+5V), LED11.3 (+5V)
- new net: LED5.4 (GND), LED6.1 (GND)
- new net: LED5.5 (DO), LED6.2 (DIN)
- new net: LED5.6 (+5V), LED6.3 (+5V)
- new net: D2.1 (K), F1.1
Other:
- note added: "SOLDERED ON PROTOBOARD"
- moved on the sheet: C1, D2, F1, LED1, LED2, LED3, LED4, LED5, LED6, LED7, LED8, LED9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

Commit message: small board changes
Connections:
- net at J1.3 (Pin_3): now also C1.2; no longer C1.1
- net at D2.2 (A), PWR_ADAPTOR1. (-PWR): now also C1.1; no longer C1.2
Changed lines of the file:
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@@
+	(wire
+		(pts
+			(xy 162.56 87.63) (xy 176.53 87.63)
+		)
+		(stroke
+			(width 0)
+			(type default)
+		)
+	)
 	(wire
 		(pts
@@
 		(pts
 			(xy 106.68 60.96) (xy 95.25 60.96)
-		)
-		(stroke
-			(width 0)
-			(type default)
-		)
-	)
-	(wire
-		(pts
-			(xy 162.56 87.63) (xy 176.53 87.63)
 		)
 		(stroke
@@
 	(symbol
 		(lib_id "Device:C_Small_US")
-		(at 173.99 78.74 0)
-		(mirror x)
+		(at 191.77 60.96 0)
+		(mirror y)
 		(unit 1)
 		(body_style 1)
@@
 		(dnp no)
 		(property "Reference" "C1"
-			(at 184.15 73.152 0)
+			(at 181.61 72.898 0)
 			(show_name no)
 			(do_not_autoplace no)
@@
 		)
 		(property "Value" "500-1000 uF"
-			(at 189.484 75.184 0)
+			(at 177.038 75.184 0)
 			(show_name no)
 			(do_not_autoplace no)
@@
 		)
 		(property "Footprint" ""
-			(at 173.99 78.74 0)
+			(at 191.77 60.96 0)
 			(hide yes)
 			(show_name no)
@@
 		)
 		(property "Datasheet" ""
-			(at 173.99 78.74 0)
+			(at 191.77 60.96 0)
 			(hide yes)
 			(show_name no)
@@
 		)
 		(property "Description" "capacitor, small US symbol"
-			(at 173.99 78.74 0)
-			(hide yes)
-			(show_name no)
+			(at 191.77 60.96 0)
+			(hide yes)
+			(show_name no)
