File: KiCAD/aviationAirportLEDMap/aviationAirportLEDMap.kicad_sch (KiCad schematic)
At the start: 20 parts, among them J1 Screw_Terminal_01x03, J2 Screw_Terminal_01x03

Commit message: Final push. Project is done and hanging on the wall.
Parts:
- removed C1: 500-1000 uF, symbol Device:C_Small_US
- removed R1: 300-900Ω, symbol Device:R_US
Connections:
- net at J1.2 (Pin_2): now also J2.5 (Pin_1)
- net at J1.3 (Pin_3): now also D2.2 (A), PWR_ADAPTOR1. (-PWR)
Other:
- moved on the sheet: D2, F1
